File: PCB/MiniQuad0/MiniQuad0.kicad_sch (KiCad schematic)
At the start: 0 parts

Commit message: schematics finish r1
Parts:
- added J1: R8EF_Radio, Connector_PinHeader_2.54mm:PinHeader_1x03_P2.54mm_Vertical, symbol Connector_Generic:Conn_01x03
- added J2: MPU6500, Connector_PinHeader_2.54mm:PinHeader_1x10_P2.54mm_Vertical, symbol Connector_Generic:Conn_01x10
- added J3: ESC_A, Connector_PinHeader_2.54mm:PinHeader_1x03_P2.54mm_Vertical, symbol Connector_Generic:Conn_01x03
- added J4: ESC_B, Connector_PinHeader_2.54mm:PinHeader_1x03_P2.54mm_Vertical, symbol Connector_Generic:Conn_01x03
- added J5: ESC_C, Connector_PinHeader_2.54mm:PinHeader_1x03_P2.54mm_Vertical, symbol Connector_Generic:Conn_01x03
- added J6: ESC_D, Connector_PinHeader_2.54mm:PinHeader_1x03_P2.54mm_Vertical, symbol Connector_Generic:Conn_01x03
- added J7: POWER, Connector_PinHeader_2.54mm:PinHeader_1x02_P2.54mm_Vertical, symbol Connector_Generic:Conn_01x02
- added J8: VBAT, Connector_PinHeader_2.54mm:PinHeader_1x01_P2.54mm_Vertical, symbol Connector_Generic:Conn_01x01
- added J9: RADIO_SIG, Connector_PinHeader_2.54mm:PinHeader_1x01_P2.54mm_Vertical, symbol Connector_Generic:Conn_01x01
- added Q1: 2N2219, Connector_PinHeader_2.54mm:PinHeader_1x03_P2.54mm_Vertical, symbol Transistor_BJT:2N2219
- added R1, R3: 10k, Connector_PinHeader_2.54mm:PinHeader_1x02_P2.54mm_Vertical, symbol Device:R_Small
- added R2, R4: 1k, Connector_PinHeader_2.54mm:PinHeader_1x02_P2.54mm_Vertical, symbol Device:R_Small
- added U2: XIAO-RP2350-SMD, Seeed Studio XIAO Series Library:XIAO-RP2350-DIP, symbol Seeed_Studio_XIAO_Series:XIAO-RP2350-SMD
Connections:
- new net: J8.1 (Pin_1), R3.2
- new net: Q1.2 (B), R2.2
- new net +3.3V: J2.10 (Pin_10), R1.1, U2.12 (3V3)
- new net +5V: J1.2 (Pin_2), J7.2 (Pin_2), U2.14 (5V)
- new net BAT_SENSE: R3.1, R4.2, U2.1 (GPIO26/D0/ADC0)
- new net GND: J1.1 (Pin_1), J2.9 (Pin_9), J3.2 (Pin_2), J4.2 (Pin_2), J5.2 (Pin_2), J6.2 (Pin_2), J7.1 (Pin_1), Q1.1 (E), R4.1, U2.13 (GND), U2.30 (GND_2)
- new net IMU_INT: J2.3 (Pin_3), U2.22 (GPIO9/D18/SPI1_CS)
- new net IMU_SCL: J2.8 (Pin_8), U2.9 (GPIO2/D8/SPI0_SCK)
- new net IMU_SD0: J2.4 (Pin_4), U2.10 (GPIO4/D9/SPI0_MISO)
- new net IMU_SDA: J2.7 (Pin_7), U2.11 (GPIO3/D10/SPI0_MOSI)
- new net MOTOR_A: J3.1 (Pin_1), U2.2 (GPIO27/D1/ADC1)
- new net MOTOR_B: J4.1 (Pin_1), U2.3 (GPIO28/D2/ADC2)
- new net MOTOR_C: J5.1 (Pin_1), U2.4 (GPIO5/D3/SPI0_CS)
- new net MOTOR_D: J6.1 (Pin_1), U2.5 (GPIO6/D4/SDA1)
- new net R8EF_SBUS: J1.3 (Pin_3), R2.1
- new net RADIO_SIG: J9.1 (Pin_1), Q1.3 (C), R1.2, U2.21 (GPIO10/D17/SPI1_SCK)
- no-connect marks 0 -> 8
Other:
- note added: "5V GND"
- note added: "5V GND SIG"
- note added: "BAT_MEASURE"
- note added: "ESCs"
- note added: "IMU"
- note added: "MCU"
- note added: "POWER_IN"
- note added: "RADIO RECEIVER"
- note added: "VCC GND SCL SDA EDA ECL AD0 INT NCS FSYNC"
- note added: "esc's bec unused as some might not have a bec and we already have bec in our pd board"
- note added: "make sure to not connect USB while battery is connected!!!"
- note added: "might need to invert in software"

Commit message: schematics update, pcb layout r2
Parts:
- removed J2: MPU6500, Connector_PinHeader_2.54mm:PinHeader_1x10_P2.54mm_Vertical, symbol Connector_Generic:Conn_01x10
- added C1, C2: 100nF, Capacitor_SMD:C_0603_1608Metric_Pad1.08x0.95mm_HandSolder, symbol Device:C_Small
- added H1, H2, H3, H4: MountingHole, MountingHole:MountingHole_3mm, symbol Mechanical:MountingHole
- added J10: BMP280_breakout, Connector_PinHeader_2.54mm:PinHeader_1x06_P2.54mm_Vertical, symbol Connector_Generic:Conn_01x06
- added J11: HMC5883L_breakout, Connector_PinHeader_2.54mm:PinHeader_1x05_P2.54mm_Vertical, symbol Connector_Generic:Conn_01x05
- added J12: MAG_drdy, TestPoint:TestPoint_Pad_D1.0mm, symbol Connector_Generic:Conn_01x01
- added J13: BAR_CSB, TestPoint:TestPoint_Pad_D1.0mm, symbol Connector_Generic:Conn_01x01
- added J14: BAR_SD0, TestPoint:TestPoint_Pad_D1.0mm, symbol Connector_Generic:Conn_01x01
- added J15: MCU_BOOT, TestPoint:TestPoint_Pad_D1.0mm, symbol Connector_Generic:Conn_01x01
- added J16: MCU_RST, TestPoint:TestPoint_Pad_D1.0mm, symbol Connector_Generic:Conn_01x01
- added J17: MCU_SWDIO, TestPoint:TestPoint_Pad_D1.0mm, symbol Connector_Generic:Conn_01x01
- added J2: POWER, Connector_PinHeader_2.54mm:PinHeader_1x03_P2.54mm_Vertical, symbol Connector_Generic:Conn_01x03
- added U1: LSM6DSOTR, easyeda2kicad:LGA-14_L3.0-W2.5-P0.50-TL, symbol easyeda2kicad:LSM6DSOTR
- J9: footprint Connector_PinHeader_2.54mm:PinHeader_1x01_P2.54mm_Vertical -> TestPoint:TestPoint_Pad_D1.0mm
- Q1: value 2N2219 -> 2N2222; footprint Connector_PinHeader_2.54mm:PinHeader_1x03_P2.54mm_Vertical -> Package_TO_SOT_SMD:TSOT-23_HandSoldering
- R1, R2, R3, R4: footprint Connector_PinHeader_2.54mm:PinHeader_1x02_P2.54mm_Vertical -> Resistor_SMD:R_1206_3216Metric_Pad1.30x1.75mm_HandSolder
- U2: footprint Seeed Studio XIAO Series Library:XIAO-RP2350-DIP -> Seeed Studio XIAO Series Library:XIAO-RP2350-SMD
Connections:
- net IMU_INT is gone; now on net RADIO_SIG: U2.22 (GPIO9/D18/SPI1_CS)
- net +3.3V: now also C1.1, C2.1, J10.6 (Pin_6), J11.1 (Pin_1), J2.2 (Pin_2), U1.2 (SDX), U1.3 (SCX), U1.5 (VDDIO), U1.8 (VDD)
- net +5V: now also J2.3 (Pin_3)
- net GND: now also U2.27 (GND_1), C1.2, C2.2, J10.5 (Pin_5), J11.2 (Pin_2), J2.1 (Pin_1), U1.6 (GND), U1.7 (GND)
- net IMU_SCL: now also U1.13 (SCL)
- net IMU_SD0: now also U2.6 (GPIO7/D5/SCL1), U1.1 (SDO/SA0)
- net IMU_SDA: now also U1.14 (SDA)
- net RADIO_SIG: no longer U2.21 (GPIO10/D17/SPI1_SCK)
- net IMU_I2C_SCL: now reaches U2.17 (GPIO17/D13/SCL0)
- net IMU_I2C_SCL: now also J10.4 (Pin_4), J11.3 (Pin_3)
- net IMU_I2C_SDA: now reaches U2.18 (GPIO16/D14/SDA0)
- net IMU_I2C_SDA: now also J10.3 (Pin_3), J11.4 (Pin_4)
- net IMU_INT1: now reaches U2.20 (GPIO12/D16/SPI1_MISO)
- net IMU_INT1: now also U1.4 (INT1)
- net at U2.23 (SWDIO): now also J17.1 (Pin_1)
- net at U2.24 (RST): now also J16.1 (Pin_1)
- net at U2.25 (BOOT): now also J15.1 (Pin_1)
- new net: J11.5 (Pin_5), J12.1 (Pin_1)
- new net: J10.1 (Pin_1), J14.1 (Pin_1)
- new net: J10.2 (Pin_2), J13.1 (Pin_1)
- new net IMU_CS: U1.12 (CS)
- new net IMU_INT2: U1.9 (INT2), U2.21 (GPIO10/D17/SPI1_SCK)
- no-connect marks 8 -> 6
Other:
- note added: "5V 3V3 GND"
- note added: "Accelerometer / Gyro"
- note added: "Barometer"
- note added: "Magnetometer"
- note added: "POWER_OUT"
- note added: "VCC GND SCL SDA CSB SD0"
- note added: "VCC GND SCL SDA DRDY"
- note removed: "VCC GND SCL SDA EDA ECL AD0 INT NCS FSYNC"
- moved on the sheet: J1, J3, J4, J5, J6, J7, J8, J9, Q1, R1, R2, R3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

Commit message: changed pin defs, finished PCB
Connections:
- net BAT_SENSE: now also U2.2 (GPIO27/D1/ADC1); no longer U2.1 (GPIO26/D0/ADC0)
- net IMU_CS: now also U2.22 (GPIO9/D18/SPI1_CS)
- net IMU_I2C_SCL: now also U2.6 (GPIO7/D5/SCL1); no longer U2.17 (GPIO17/D13/SCL0)
- net IMU_I2C_SDA: now also U2.5 (GPIO6/D4/SDA1); no longer U2.18 (GPIO16/D14/SDA0)
- net IMU_INT1: now also U2.16 (GPIO20/D12/TX1); no longer U2.20 (GPIO12/D16/SPI1_MISO)
- net IMU_INT2: now also U2.15 (GPIO21/D11/RX1); no longer U2.21 (GPIO10/D17/SPI1_SCK)
- net IMU_SCL: now also U2.21 (GPIO10/D17/SPI1_SCK); no longer U2.9 (GPIO2/D8/SPI0_SCK)
- net IMU_SD0: now also U2.20 (GPIO12/D16/SPI1_MISO); no longer U2.10 (GPIO4/D9/SPI0_MISO), U2.6 (GPIO7/D5/SCL1)
- net IMU_SDA: now also U2.19 (GPIO11/D15/SPI1_MOSI); no longer U2.11 (GPIO3/D10/SPI0_MOSI)
- net MOTOR_A: now also U2.9 (GPIO2/D8/SPI0_SCK); no longer U2.2 (GPIO27/D1/ADC1)
- net MOTOR_B: now also U2.4 (GPIO5/D3/SPI0_CS); no longer U2.3 (GPIO28/D2/ADC2)
- net MOTOR_C: now also U2.1 (GPIO26/D0/ADC0); no longer U2.4 (GPIO5/D3/SPI0_CS)
- net MOTOR_D: now also U2.11 (GPIO3/D10/SPI0_MOSI); no longer U2.5 (GPIO6/D4/SDA1)
- net RADIO_SIG: now also U2.3 (GPIO28/D2/ADC2); no longer U2.22 (GPIO9/D18/SPI1_CS)
Changed lines of the file:
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@@
+	(wire
+		(pts
+			(xy 118.11 109.22) (xy 133.35 109.22)
+		)
+		(stroke
+			(width 0)
+			(type default)
+		)
+	)
 	(wire
 		(pts
@@
 	(wire
 		(pts
+			(xy 182.88 116.84) (xy 198.12 116.84)
+		)
+		(stroke
+			(width 0)
+			(type default)
+		)
+	)
+	(wire
+		(pts
 			(xy 182.88 93.98) (xy 186.69 93.98)
 		)
@@
 	(wire
 		(pts
+			(xy 118.11 97.79) (xy 133.35 97.79)
+		)
+		(stroke
+			(width 0)
+			(type default)
+		)
+	)
+	(wire
+		(pts
 			(xy 193.04 34.29) (xy 198.12 34.29)
 		)
@@
 	(wire
 		(pts
+			(xy 118.11 93.98) (xy 133.35 93.98)
+		)
+		(stroke
+			(width 0)
+			(type default)
+		)
+	)
+	(wire
+		(pts
 			(xy 46.99 167.64) (xy 50.8 167.64)
 		)
@@
 	(wire
 		(pts
+			(xy 182.88 120.65) (xy 198.12 120.65)
+		)
+		(stroke
+			(width 0)
+			(type default)
+		)
+	)
+	(wire
+		(pts
 			(xy 77.47 132.08) (xy 80.01 132.08)
 		)
@@
 	)
 	(label "IMU_I2C_SDA"
-		(at 118.11 105.41 0)
+		(at 198.12 128.27 180)
+		(effects
+			(font
+				(size 1.27 1.27)
+			)
+			(justify right bottom)
+		)
+	)
+	(label "IMU_INT2"
+		(at 118.11 93.98 0)
 		(effects
 			(font
@@
 	)
 	(label "IMU_SCL"
-		(at 198.12 113.03 180)
-		(effects
-			(font
-				(size 1.27 1.27)
-			)
-			(justify right bottom)
+		(at 118.11 116.84 0)
+		(effects
+			(font
+				(size 1.27 1.27)
+			)
+			(justify left bottom)
 		)
 	)
 	(label "MOTOR_C"
-		(at 198.12 132.08 180)
+		(at 198.12 143.51 180)
 		(effects
 			(font
@@
 	)
 	(label "MOTOR_A"
-		(at 198.12 139.7 180)
+		(at 198.12 113.03 180)
 		(effects
 			(font
@@
 	)
 	(label "IMU_SDA"
-		(at 198.12 105.41 180)
-		(effects
-			(font
-				(size 1.27 1.27)
-			)
-			(justify right bottom)
+		(at 118.11 109.22 0)
+		(effects
+			(font
+				(size 1.27 1.27)
+			)
+			(justify left bottom)
+		)
+	)
+	(label "IMU_CS"
+		(at 118.11 120.65 0)
+		(effects
+			(font
+				(size 1.27 1.27)
+			)
+			(justify left bottom)
 		)
 	)
 	(label "MOTOR_B"
-		(at 198.12 135.89 180)
+		(at 198.12 132.08 180)
 		(effects
 			(font
@@
 	)
 	(label "IMU_SD0"
-		(at 198.12 124.46 180)
-		(effects
-			(font
-				(size 1.27 1.27)
-			)
-			(justify right bottom)
+		(at 118.11 113.03 0)
+		(effects
+			(font
+				(size 1.27 1.27)
+			)
+			(justify left bottom)
 		)
 	)
 	(label "MOTOR_D"
-		(at 198.12 128.27 180)
+		(at 198.12 105.41 180)
 		(effects
 			(font
@@
 		)
 	)
-	(label "IMU_SD0"
-		(at 198.12 109.22 180)
-		(effects
-			(font
-				(size 1.27 1.27)
-			)
-			(justify right bottom)
-		)
-	)
-	(label "IMU_INT2"
-		(at 118.11 116.84 0)
-		(effects
-			(font
-				(size 1.27 1.27)
-			)
-			(justify left bottom)
-		)
-	)
 	(label "MOTOR_D"
 		(at 262.89 105.41 180)
@@
 	)
 	(label "BAT_SENSE"
-		(at 198.12 143.51 180)
+		(at 198.12 139.7 180)
 		(effects
 			(font
@@
 	)
 	(label "IMU_I2C_SCL"
-		(at 118.11 101.6 0)
+		(at 198.12 124.46 180)
+		(effects
+			(font
+				(size 1.27 1.27)
+			)
+			(justify right bottom)
+		)
+	)
+	(label "IMU_INT1"
+		(at 118.11 97.79 0)
 		(effects
 			(font
@@
 		)
 	)
-	(label "IMU_INT1"
-		(at 118.11 113.03 0)
-		(effects
-			(font
-				(size 1.27 1.27)
-			)
-			(justify left bottom)
-		)
-	)
 	(label "RADIO_SIG"
-		(at 118.11 120.65 0)
-		(effects
-			(font
-				(size 1.27 1.27)
-			)
-			(justify left bottom)
-		)
-	)
+		(at 198.12 135.89 180)
+		(effects
+			(font
+				(size 1.27 1.27)
+			)
+			(justify right bottom)
+		)
+	)

Commit message: added test pads for unused pins under the mcu which were inaccessible otherwise
Parts:
- added J18: MCU_SWDCLK, TestPoint:TestPoint_Pad_D1.0mm, symbol Connector_Generic:Conn_01x01
- added J19: MCU_GP17, TestPoint:TestPoint_Pad_D1.0mm, symbol Connector_Generic:Conn_01x01
- added J20: MCU_GP16, TestPoint:TestPoint_Pad_D1.0mm, symbol Connector_Generic:Conn_01x01
- added J21: MCU_GP04, TestPoint:TestPoint_Pad_D1.0mm, symbol Connector_Generic:Conn_01x01
Connections:
- net +3.3V: now also U2.26 (3V3_1)
- net at U2.10 (GPIO4/D9/SPI0_MISO): now also J21.1 (Pin_1)
- net at U2.17 (GPIO17/D13/SCL0): now also J19.1 (Pin_1)
- net at U2.18 (GPIO16/D14/SDA0): now also J20.1 (Pin_1)
- net at U2.28 (SWDCLK): now also J18.1 (Pin_1)
